File: esp32s2_devboard.kicad_sch (KiCad schematic)
At the start: 31 parts, among them J1 USB_C_Receptacle_USB2.0, J2 USB_C_Receptacle_USB2.0, J3 Conn_01x15, J4 Conn_01x15, Q1 BC817, Q2 BC817, SW1 SW_DPST, SW2 SW_DPST, U1 ESP32-S2-MINI-2, U2 AP2112K-3.3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

Commit message: Added sch scheets, project on hold
Parts:
- removed C1: 22uF, Capacitor_SMD:C_0603_1608Metric, symbol Device:C_Small
- removed C2, C5: 100n, Capacitor_SMD:C_0603_1608Metric, symbol Device:C_Small
- removed C3, C6: 1u, Capacitor_SMD:C_0603_1608Metric, symbol Device:C
- removed C4, C7: 1u, Capacitor_SMD:C_0603_1608Metric, symbol Device:C_Small
- removed D1, D2: PRTR5V0U2X, Package_TO_SOT_SMD:SOT-143, symbol Power_Protection:PRTR5V0U2X
- removed D3: GREEN, LED_SMD:LED_0603_1608Metric, symbol Device:LED
- removed F1: 500mA, Fuse:Fuse_0603_1608Metric, symbol Device:Polyfuse
- removed J1, J2: USB_C_Receptacle_USB2.0, Connector_USB:USB_C_Receptacle_HRO_TYPE-C-31-M-12, symbol Connector:USB_C_Receptacle_USB2.0
- removed J3, J4: Conn_01x15, Connector_PinHeader_2.54mm:PinHeader_1x15_P2.54mm_Vertical, symbol Connector_Generic:Conn_01x15
- removed Q1, Q2: BC817, Package_TO_SOT_SMD:SOT-23, symbol Transistor_BJT:BC817
- removed R1, R2, R3, R4: 5k1, Resistor_SMD:R_0603_1608Metric, symbol Device:R_Small
- removed R5, R7: 22k, Resistor_SMD:R_0603_1608Metric, symbol Device:R_Small
- removed R6: 3k3, Resistor_SMD:R_0603_1608Metric, symbol Device:R
- removed R8, R9: 10k, Resistor_SMD:R_0603_1608Metric, symbol Device:R_Small
- removed SW1, SW2: SW_DPST, SKRPACE010:SW_SKRPACE010, symbol Switch:SW_DPST
- removed U1: ESP32-S2-MINI-2, Espressif:ESP32-S2-MINI-1, symbol Espressif:ESP32-S2-MINI-1
- removed U2: AP2112K-3.3, Package_TO_SOT_SMD:SOT-23-5, symbol Regulator_Linear:AP2112K-3.3
- removed U3: CH340C, Package_SO:SOIC-16_3.9x9.9mm_P1.27mm, symbol Interface_USB:CH340C
Connections:
- no-connect marks 14 -> 0
Other:
- added sheet MCU (mcu.kicad_sch)
- added sheet Pheripherals (pheripherals.kicad_sch)
- added sheet Power (power.kicad_sch)
- note removed: "- GPIO46 is fixed pull-down internally, only used as 0 anyway - GPIO45 is default pull-down, used to select VDD_SPI to 3v3(0) or 1v8(1)"
- note removed: "- debounce time is R*C, 22k*1u=22 ms"
- note removed: "JTAG"
- note removed: "LDO"
- note removed: "MCU"
- note removed: "NOTE: LDO is 600mA max"
- note removed: "Reset, GPIO0"
- note removed: "USB OTG"
- note removed: "USB-UART bridge, ESD"
